File: kicad/civil25.kicad_sch (KiCad schematic)
At the start: 8 parts, among them U1 8088_Min_Mode, U2 SST39SF020, U3 AS6C4008-55PCN, U4 74HC245, U5 74HC373, U6 74HC373, U7 74HCT238, U8 74HC00

Commit message: remove unused assemblers/update gcc
Connections:
- net A0: no longer U3.22 (CE#)
- net A19: now also U3.22 (CE#)
Changed lines of the file:
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@@
     (effects (font (size 1.27 1.27)) (justify left bottom))
   )
-  (label "A0" (at 218.44 135.89 0)
+  (label "A19" (at 218.44 135.89 0)
     (effects (font (size 1.27 1.27)) (justify left bottom))
   )
@@
     (pin "2")
     (pin "3")
-    (pin "4")
-    (pin "5")
-    (pin "6")
-    (pin "10")
-    (pin "8")
-    (pin "9")
-    (pin "11")
-    (pin "12")
-    (pin "13")
-    (pin "14")
-    (pin "7")
   )
   (symbol (lib_id "74xx:74HCT238") (at 123.19 166.37 0) (unit 1)

Commit message: update PCB
Parts:
- removed U8: 74HC00, Package_DIP:DIP-14_W7.62mm_Socket, symbol 74xx:74HC00
- added RV1: 10k, Potentiometer_THT:Potentiometer_ACP_CA9-V10_Vertical, symbol Device:R_Potentiometer
- added U10: LCD-016N002L, Display:WC1602A, symbol Display_Character:LCD-016N002L
- added U11: 74LS138, Package_DIP:DIP-16_W7.62mm_Socket, symbol 74xx:74LS138
- added U14: 74LS10, Package_DIP:DIP-14_W7.62mm_Socket, symbol 74xx:74LS10
- added U18: TL072, Package_DIP:DIP-8_W7.62mm_Socket, symbol Amplifier_Operational:TL072
- added U9: 82C55A, Package_DIP:DIP-40_W15.24mm, symbol Interface:82C55A
Connections:
- net +5V: now also RV1.1, U10.15 (A/VEE), U10.2 (VDD), U11.16 (VCC), U11.6 (E3), U18.8 (V+), U9.26 (VCC)
- net A0: now also U9.9 (A0)
- net A1: now also U9.8 (A1)
- net A18: now also U14.1
- net A19: now also U14.13
- net A4: now also U11.1 (A0)
- net A5: now also U11.2 (A1)
- net A6: now also U11.3 (A2)
- net CE_ROM: now also U14.12
- net D0: now also U9.34 (D0)
- net D1: now also U9.33 (D1)
- net D2: now also U9.32 (D2)
- net D3: now also U9.31 (D3)
- net D4: now also U9.30 (D4)
- net D5: now also U9.29 (D5)
- net D6: now also U9.28 (D6)
- net D7: now also U9.27 (D7)
- net GND: now also U10.1 (VSS), U10.16 (K), U11.4 (E1), U11.5 (E2), U11.8 (GND), U18.4 (V-), U9.7 (GND); no longer U1.18 (INTR), U1.34 (~{SSO})
- net CLK: now reaches U1.19 (CLK)
- net RESET: now reaches U1.21 (RESET)
- net RESET: now also U9.35 (RESET)
- net READY: now reaches U1.22 (READY)
- net A16/S3 renamed S3
- net A17/S4 renamed S4
- net A18/S5 renamed S5
- net A19/S6 renamed S6
- net IO/M renamed RD/
- net RD/: now also U9.36 (~{WR}), U9.5 (~{RD})
- net RD renamed IO/M/
- net IO/M/: now also U14.2
- new net: U10.10 (DB3), U9.1 (PA3)
- new net: U10.9 (DB2), U9.2 (PA2)
- new net: U10.8 (DB1), U9.3 (PA1)
- new net: U10.14 (DB7), U9.37 (PA7)
- new net: U10.13 (DB6), U9.38 (PA6)
- new net: U10.12 (DB5), U9.39 (PA5)
- new net: U10.7 (DB0), U9.4 (PA0)
- new net: U10.11 (DB4), U9.40 (PA4)
- new net: RV1.2, U10.3 (VO)
- new net INTR: U1.18 (INTR)
- new net IO_DEVICE0/: U11.15 (O0), U9.6 (~{CS})
- new net IO_DEVICE1/: U11.14 (O1)
- new net IO_DEVICE2/: U11.13 (O2)
- new net IO_DEVICE3/: U11.12 (O3)
- new net IO_DEVICE4/: U11.11 (O4)
- new net IO_DEVICE5/: U11.10 (O5)
- new net IO_DEVICE6/: U11.9 (O6)
- new net IO_DEVICE7/: U11.7 (O7)
- new net PB0: U10.6 (E), U9.18 (PB0)
- new net PB1: U10.5 (R/~{W}), U9.19 (PB1)
- new net PB2: U10.4 (RS), U9.20 (PB2)
- no-connect marks 13 -> 19
Other:
- added sheet CLK (untitled.kicad_sch)
- added sheet POWER (power.kicad_sch)
- added sheet YM3812 (ym3812.kicad_sch)
- note added: "NOTE: WR IS ALSO ACTIVE LOW"
- moved on the sheet: U1, U2, U3, U4, U5, U6, U7
